Commit message: fixed up some urdf stuff, did some more testing. looking good. unsure of coord sys conventions in urdf

File: urdf/modleg.urdf (robot description, URDF)
Before this commit: robot Modular Leg, 6 links, 5 joints
Links:
- removed link Foot_link
- added link foot_link, mass 0.0047851; collision mesh filename=package://Fourth_URDF_test.urdf/meshes/foot_link.STL; visual mesh filename=package://Fourth_URDF_test.urdf/meshes/foot_link.STL
Joints:
- removed joint Ankle Joint
- removed joint base_to_femur
- added joint ankle_joint: type revolute, parent tibia_link, child podial_link, origin xyz=0.000 0.140 -0.025 rpy=0 0 0, axis -1 0 0, limit lower=-0.9076 upper=1.1868 effort=0 velocity=0
- added joint hip_joint: type continuous, parent base_link, child femur_link, origin xyz=-0.1116 0 0 rpy=0 0 0, axis 1 0 0, limit lower=0 upper=0 effort=0 velocity=0
- joint knee_joint: origin xyz=0.02414 0 -0.12699 rpy=0 0 0 -> xyz=0.025 0.000 -0.125 rpy=0 0 0
- joint tibia_to_foot: child Foot_link -> foot_link; origin xyz=0 0.01800 -0.1350 rpy=0 0 0 -> xyz=0.000 0.018 -0.135 rpy=0 0 0

Commit message: drafted kinematics

File: urdf/modleg.urdf (robot description, URDF)
Before this commit: robot Modular Leg, 6 links, 5 joints
Joints:
- removed joint tibia_to_foot
- added joint tibia_foot_joint: type fixed, parent podial_link, child foot_link, origin xyz=0.000 0.018 -0.135 rpy=0 0 0, axis 0 0 0
